Commit message: Changed orientation of all camera frames to be equal to the color cam frame

File: urdf/realsense-RS200.macro.xacro (robot description, xacro)
@@ -59,15 +59,15 @@
         <parent link="${prefix}rs200_camera" />
         <child link="${prefix}depth" />
-        <origin xyz="0 -0.03 0.004" rpy="0 0 0"/>
+        <origin xyz="0 -0.03 0.004" rpy="${pi/2} ${pi} ${pi/2}"/>
     </joint>
     <joint name="${prefix}ired1_joint" type="fixed">
         <parent link="${prefix}rs200_camera" />
         <child link="${prefix}ired1" />
-        <origin xyz="0 -0.06 0.004" rpy="0 0 0"/>
+        <origin xyz="0 -0.06 0.004" rpy="${pi/2} ${pi} ${pi/2}"/>
     </joint>
     <joint name="${prefix}ired2_joint" type="fixed">
         <parent link="${prefix}rs200_camera" />
         <child link="${prefix}ired2" />
-        <origin xyz="0 0.01 0.004" rpy="0 0 0"/>
+        <origin xyz="0 0.01 0.004" rpy="${pi/2} ${pi} ${pi/2}"/>
     </joint>
 <!-- **********************************************************-->
@@ -98,6 +98,6 @@
             <horizontal_fov>1.047</horizontal_fov>
             <image>
-                <width>640</width>
-                <height>480</height>
+                <width>1280</width>
+                <height>960</height>
                 <format>R8G8B8</format>
             </image>
